File: STEC_Design.kicad_sch (KiCad schematic)
At the start: 13 parts, among them Q1 IRLB3034PBF, Q2 IRLB3034PBF, SW1 SW_Push, SW2 SW_Push, U1 L7805CV, U2 MLX90614ESF-BAA-000-TU, U3 ESP32-WROOM-32E

Commit message: added_ESP32_DevBoard
Parts:
- added U4: ESP32-DEVKITC-32E, footprints:MODULE_ESP32-DEVKITC-32E, symbol ESP32-DEVKITC-32E:ESP32-DEVKITC-32E
- BT1: footprint (none) -> Connector_Wire:SolderWire-0.5sqmm_1x02_P4.8mm_D0.9mm_OD2.3mm
- D1, D2: footprint (none) -> LED_THT:LED_D5.0mm
- PE1: footprint (none) -> Connector_Wire:SolderWire-0.75sqmm_1x02_P7mm_D1.25mm_OD3.5mm
- Q1, Q2: footprint Package_TO_SOT_THT:TO-220-3_Vertical -> IRLB3034PBF:TO254P1041X444X1930-3
- R1, R2: footprint (none) -> Resistor_THT:R_Axial_DIN0309_L9.0mm_D3.2mm_P12.70mm_Horizontal
- SW1, SW2: footprint (none) -> Button_Switch_THT:SW_PUSH_6mm_H4.3mm
- U1: footprint (none) -> Package_TO_SOT_THT:TO-220-3_Vertical
Connections:
- net GND: now also U4.J2_14 (GND_J2_14)

Commit message: finalisedSchematics
Parts:
- removed U3: ESP32-WROOM-32E, RF_Module:ESP32-WROOM-32D, symbol RF_Module:ESP32-WROOM-32E
- SW1: value SW_Push -> SW_Push (Down)
- SW2: value SW_Push -> SW_Push (Up)
Connections:
- net GND: no longer U4.J2_14 (GND_J2_14)
- net at U1.3 (OUT), U2.3 (VDD): now also U4.J2_19 (EXT_5V)
- net at SW1.1: now also U4.J3_13 (IO4)
- net at SW2.1: now also U4.J3_10 (IO5)
- net at Q1.1 (G), Q2.1 (G): now also U4.J3_9 (IO18)
- net at U2.2 (SDA/PWM): now also U4.J3_6 (IO21)
- net at U2.1 (SCL/VZ): now also U4.J3_3 (IO22)
- net at R2.2: now also U4.J3_2 (IO23)
- no-connect marks 21 -> 31
Other:
- moved on the sheet: D1, D2, Q1, R1, R2, SW1, SW2, U2, U4

Commit message: finishedPCBdesign
Parts:
- added PE2, PE3: TEC, Connector_Wire:SolderWire-0.75sqmm_1x02_P7mm_D1.25mm_OD3.5mm, symbol Device:PeltierElement
- D2: value WiFi_LED -> WiFi_LED (Red)
- PE1: value TEC(x3) -> TEC
Connections:
- net +12V: now also PE2.2, PE3.2
- net GND: now also Q1.3 (S), Q2.3 (S), U4.J2_14 (GND_J2_14), U4.J3_1 (GND_J3_1), U4.J3_7 (GND_J3_7); no longer Q1.2 (D), Q2.2 (D)
- net at D1.1 (K), PE1.1: now also Q1.2 (D), Q2.2 (D), PE2.1, PE3.1; no longer Q1.3 (S), Q2.3 (S)
- net +5V: now reaches U1.3 (OUT), U2.3 (VDD), U4.J2_19 (EXT_5V)
- no-connect marks 31 -> 28
Other:
- moved on the sheet: Q1

Commit message: BeforePotentiometer
Parts:
- added C1: C_Polarized (10 μF), Capacitor_THT:CP_Radial_D5.0mm_P2.00mm, symbol Device:C_Polarized
- added C2, C3, C5: C (0.1 μF), Capacitor_THT:C_Disc_D4.3mm_W1.9mm_P5.00mm, symbol Device:C
- added C4: C (0.33 μF), Capacitor_THT:C_Disc_D4.3mm_W1.9mm_P5.00mm, symbol Device:C
Connections:
- net +12V: now also C1.1, C4.1
- net +5V: now also C2.2, C3.2, C5.2
- net GND: now also C1.2, C2.1, C3.1, C4.2, C5.1
Other:
- moved on the sheet: BT1, D1, D2, PE1, PE2, PE3, Q1, R1, R2, SW1, SW2, U1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
